File: pcb/octoboard.kicad_pcb (KiCad board)
At the start: 2 copper layers, 45 x 74.5 mm, 29 parts, among them J1 ICSP, J2 Serial Board, J3 Conn_01x08, J4 Conn_01x06, J5 Conn_01x06, J6 Conn_01x04, J7 Barrel_Jack, J8 Conn_01x02, SW1 SW_Push, U1 ATmega328P-P, U2 LM7805_TO220, Y1 Crystal

Commit message: Added some mounting holes
how tf did i forget that
Parts:
- added H1: MountingHole, MountingHole:MountingHole_2.2mm_M2, F.Cu at (101.5, 119.0)
- added H2: MountingHole, MountingHole:MountingHole_2.2mm_M2, F.Cu at (134.5, 119.0)
- added H3: MountingHole, MountingHole:MountingHole_2.2mm_M2, F.Cu at (134.5, 49.5)
Routing:
- net GND: vias 21 -> 25
