File: pcb/octoboard.kicad_sch (KiCad schematic)
At the start: 27 parts, among them J1 Conn_02x03_Odd_Even, J2 Conn_01x06, J3 Conn_01x08, J4 Conn_01x06, J5 Conn_01x06, J6 Conn_01x04, J7 Barrel_Jack, J8 Conn_01x02, SW1 SW_Push, U1 ATmega328P-P, U2 LM7805_TO220, Y1 Crystal

Commit message: Added some mounting holes
how tf did i forget that
Parts:
- added H1, H2, H3: MountingHole, MountingHole:MountingHole_2.2mm_M2, symbol Mechanical:MountingHole
- C7: value 47uF, 25V -> 47uF
- C8: value 47uf, 25V -> 47uf
- J1: value Conn_02x03_Odd_Even -> ICSP
- J2: value Conn_01x06 -> Serial Board
Other:
- note added: "Mounting Holes"
